File: hw/utrak.sch (EAGLE design)
At the start: 46 parts, among them IC1 SI4060, Q1 BLAH, U1 TLV61225

Commit message: add new hardware files
Parts:
- removed AAA+, AAA-: (no value), wirepad:SMD2
- removed C1: 10u, rcl:C-EUC1210
- removed C13: 560p, rcl:C-EUC0603
- removed C14: 12p, rcl:C-EUC0603
- removed C2: 10u, rcl:C-EUC1206
- removed D1: (no value), diode:DIODE_CAPACITANCE-SOD523
- removed L1: 4u7, l2424:L2424
- removed LED1: (no value), led:LEDSML0603
- removed R3: 470, rcl:R-EU_R0603
- removed U1: TLV61225, texas_ureg:TLV61225
- added C8: 8p2, rcl:C-EUC0402
- added JP2: (no value), pinhead:PINHD-1X3
- added R6, R7: 0, rcl:R-EU_R0402
- added TP10, TP11, TP9: PTR1TP07R, testpad:PTR1TP07R
- GPS1: value RXM-GPS-RM-B -> MAX-7; device gps-linx:RXM-GPS-RM-B -> ublox-gps:MAX-7
- R1, R2: device rcl:R-EU_R0603 -> rcl:R-EU_R0402
- R4: value 220k -> 0; device rcl:R-EU_R0603 -> rcl:R-EU_R0402
- R5: value 2M -> 0; device rcl:R-EU_R0603 -> rcl:R-EU_R0402
Connections:
- net XO_MOD renamed XO_EN
- removed net N$1: L1.2, U1.L
- removed net VAAA: AAA+.P, C1.1, L1.1, U$1.P1.2/A2, U1.EN, U1.VIN
- new net ADC_IN: JP2.2, U$1.P1.2/A2
- net +3V3: now also GPS1.!RESET, GPS1.VCC_BK, GPS1.VCC_IO, JP2.3, R6.1, TP10.TP; no longer C2.1, GPS1.VBAT, U1.FB, U1.VOUT
- net GND: now also GPS1.GND, JP2.1, R7.1, TP11.TP; no longer AAA-.P, C1.2, C13.2, C2.2, D1.A, GPS1.GND@3, GPS1.GND@4, Q1.4, TP3.TP, U1.GND
- net GPS_ANT_+: now also GPS1.RF_IN; no longer GPS1.RFIN
- net LED_A: now also TP9.TP; no longer LED1.A
- net LED_K: now also TP3.TP; no longer R3.2
- net N$11: now also Q1.4, R6.2, R7.2; no longer IC1.XIN, Q1.1
- net N$12: now also C8.1, Q1.3; no longer C14.2, D1.C, R5.1
- net N$13: now also IC1.XOUT; no longer C13.1, R4.1
- net N$14: now also C8.2, IC1.XIN; no longer C14.1, IC1.XOUT, Q1.3
- net N$8: now also Q1.1, R4.1, R5.1; no longer LED1.C, R3.1
Other:
- note removed: "LED"
- note removed: "LED anode and cathode to MSP430 for light-sensing, signalling, comms.."
- note removed: "Pads for AAA"
- note removed: "Power Supply"
- note removed: "antenna = 2x 5cm guitar string, 2 PADs"
- note removed: "optional"
- moved on the sheet: GPS_ANT_+, Q1, R4, R5, TP3, TP4, TP5, TP6, TP7, TP8
